File: distribution-5v/distribution-5v.kicad_pcb (KiCad board)
At the start: 2 copper layers, 35 x 60 mm, 11 parts, among them J1 Conn_01x02_Socket, J2 Conn_01x02_Socket, J3 Conn_01x02_Socket, J4 Conn_01x02_Socket, J5 Conn_01x02_Socket

Commit message: feat: 寸法を追加
Other:
- board text added: "※6Aまで"
- board text added: "配電基盤 (5V) v1"
- board text removed: "※5V 20Aまで"
- board text removed: "分電基盤"
Changed lines of the file:
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@@
 		(tags "RC Connector XT30")
 		(property "Reference" "J3"
-			(at 2.5 -4 360)
+			(at 2.5 -4 0)
 			(layer "F.SilkS")
 			(effects
@@
 		)
 		(property "Value" "Conn_01x02_Socket"
-			(at 2.5 4 360)
+			(at 2.5 4 0)
 			(layer "F.Fab")
 			(effects
@@
 		)
 		(fp_text user "+"
-			(at 9 0 360)
+			(at 9 0 0)
 			(layer "F.SilkS")
 			(effects
@@
 		)
 		(fp_text user "-"
-			(at -4 0 360)
+			(at -4 0 0)
 			(layer "F.SilkS")
 			(effects
@@
 		)
 		(fp_text user "${REFERENCE}"
-			(at 2.5 0 360)
+			(at 2.5 0 0)
 			(layer "F.Fab")
 			(effects
@@
 		(property "Reference" "H2"
 			(at 0 -4.2 0)
-			(layer "F.SilkS")
+			(layer "F.Fab")
 			(effects
 				(font
@@
 		(property "Reference" "H3"
 			(at 0 -4.2 0)
-			(layer "F.SilkS")
+			(layer "F.Fab")
 			(effects
 				(font
@@
 		(property "Reference" "H4"
 			(at 0 -4.2 0)
-			(layer "F.SilkS")
+			(layer "F.Fab")
 			(effects
 				(font
@@
 		(property "Value" "120Ω"
 			(at 5.08 2.37 90)
-			(layer "F.Fab")
+			(layer "F.SilkS")
 			(effects
 				(font
@@
 			(layer "F.Fab")
 		)
+		(fp_text user "${REFERENCE}"
+			(at -2.5 -3 0)
+			(layer "F.SilkS")
+			(effects
+				(font
+					(size 1 1)
+					(thickness 0.15)
+				)
+			)
+		)
 		(fp_text user "-"
 			(at 3 0 0)
@@
 				(font
 					(size 1.5 1.5)
-					(thickness 0.15)
-				)
-			)
-		)
-		(fp_text user "${REFERENCE}"
-			(at -2.5 -3 0)
-			(layer "F.Fab")
-			(effects
-				(font
-					(size 1 1)
 					(thickness 0.15)
 				)
@@
 		(tags "RC Connector XT30")
 		(property "Reference" "J5"
-			(at 2.5 -4 360)
+			(at 2.5 -4 0)
 			(layer "F.SilkS")
 			(effects
@@
 		)
 		(property "Value" "Conn_01x02_Socket"
-			(at 2.5 4 360)
+			(at 2.5 4 0)
 			(layer "F.Fab")
 			(effects
@@
 		)
 		(fp_text user "+"
-			(at 9 0 360)
+			(at 9 0 0)
 			(layer "F.SilkS")
 			(effects
@@
 		)
 		(fp_text user "-"
-			(at -4 0 360)
+			(at -4 0 0)
 			(layer "F.SilkS")
 			(effects
@@
 		)
 		(fp_text user "${REFERENCE}"
-			(at 2.5 0 360)
+			(at 2.5 0 0)
 			(layer "F.Fab")
 			(effects
@@
 		(property "Reference" "H1"
 			(at 0 -4.2 0)
-			(layer "F.SilkS")
+			(layer "F.Fab")
 			(effects
 				(font
@@
 		(tags "LED diameter 5.0mm 2 pins")
 		(property "Reference" "D1"
-			(at 1.27 -3.96 360)
+			(at 1.5 4 0)
 			(layer "F.SilkS")
 			(effects
@@
 		)
 		(property "Value" "LED"
-			(at 1.27 3.96 360)
+			(at 1.5 6 0)
 			(layer "F.Fab")
 			(effects
@@
 		)
 		(fp_text user "${REFERENCE}"
-			(at 1.25 0 360)
+			(at 1.25 0 0)
 			(layer "F.Fab")
 			(effects
@@
 		(tags "RC Connector XT30")
 		(property "Reference" "J4"
-			(at 2.5 -4 360)
+			(at 2.5 -4 0)
 			(layer "F.SilkS")
 			(effects
@@
 		)
 		(property "Value" "Conn_01x02_Socket"
-			(at 2.5 4 360)
+			(at 2.5 4 0)
 			(layer "F.Fab")
 			(effects
@@
 		)
 		(fp_text user "-"
-			(at -4 0 360)
+			(at -4 0 0)
 			(layer "F.SilkS")
 			(effects
@@
 		)
 		(fp_text user "+"
-			(at 9 0 360)
+			(at 9 0 0)
 			(layer "F.SilkS")
 			(effects
@@
 		)
 		(fp_text user "${REFERENCE}"
-			(at 2.5 0 360)
+			(at 2.5 0 0)
 			(layer "F.Fab")
 			(effects
@@
 		(tags "RC Connector XT30")
 		(property "Reference" "J2"
-			(at 2.5 -15.5 360)
+			(at 2.5 -15.5 0)
 			(layer "F.SilkS")
 			(effects
@@
 		)
 		(property "Value" "Conn_01x02_Socket"
-			(at 2.5 3.5 360)
+			(at 2.5 3.5 0)
 			(layer "F.Fab")
 			(effects
@@
 			(layer "F.Fab")
 		)
+		(fp_text user "${REFERENCE}"
+			(at 2.5 -3 0)
+			(layer "F.SilkS")
+			(effects
+				(font
+					(size 1 1)
+					(thickness 0.15)
+				)
+			)
+		)
 		(fp_text user "-"
-			(at -3 0 360)
+			(at -3 0 0)
 			(layer "F.SilkS")
 			(effects
@@
 		)
 		(fp_text user "+"
-			(at 8 0 360)
+			(at 8 0 0)
 			(layer "F.SilkS")
 			(effects
 				(font
 					(size 1.5 1.5)
-					(thickness 0.15)
-				)
-			)
-		)
-		(fp_text user "${REFERENCE}"
-			(at 2.5 -3 360)
-			(layer "F.Fab")
-			(effects
-				(font
-					(size 1 1)
 					(thickness 0.15)
 				)
@@
 	)
 	(gr_text "新居浜高専"
-		(at 163 68 270)
+		(at 163 67 270)
 		(layer "F.SilkS")
 		(effects
@@
 		)
 	)
-	(gr_text "※5V 20Aまで"
-		(at 161 78 270)
+	(gr_text "※6Aまで"
+		(at 160 88 270)
 		(layer "F.SilkS")
 		(effects
@@
 		)
 	)
-	(gr_text "分電基盤"
-		(at 161 68 270)
+	(gr_text "配電基盤 (5V) v1"
+		(at 160 68 270)
 		(layer "F.SilkS")
 		(effects
@@
 			(justify left bottom)
 		)
+	)
+	(dimension
+		(type aligned)
+		(layer "Dwgs.User")
+		(pts
+			(xy 137.5 60) (xy 162.5 60)
+		)
+		(height -12)
+		(gr_text "25.0000 mm"
+			(at 150 46.85 0)
+			(layer "Dwgs.User")
+			(effects
+				(font
+					(size 1 1)
+					(thickness 0.15)
+				)
+			)
+		)
+		(format
+			(prefix "")
+			(suffix "")
+			(units 3)
+			(units_format 1)
+			(precision 4)
+		)
+		(style
+			(thickness 0.1)
+			(arrow_length 1.27)
+			(text_position_mode 0)
+			(extension_height 0.58642)
+			(extension_offset 0.5) keep_text_aligned)
+	)
+	(dimension
+		(type aligned)
+		(layer "Dwgs.User")
+		(pts
+			(xy 137.5 60) (xy 137.5 110)
+		)
+		(height 14.5)
+		(gr_text "50.0000 mm"
+			(at 121.85 85 90)
+			(layer "Dwgs.User")
+			(effects
+				(font
+					(size 1 1)
+					(thickness 0.15)
+				)
+			)
+		)
+		(format
+			(prefix "")
+			(suffix "")
+			(units 3)
+			(units_format 1)
+			(precision 4)
+		)
+		(style
+			(thickness 0.1)
+			(arrow_length 1.27)
+			(text_position_mode 0)
+			(extension_height 0.58642)
+			(extension_offset 0.5) keep_text_aligned)
 	)
 	(dimension
@@
 		(priority 1)
 		(connect_pads yes
-			(clearance 1)
+			(clearance 1.25)
 		)
 		(min_thickness 0.25)
@@
 		(polygon
 			(pts
-				(xy 149 66) (xy 148 65) (xy 138 65) (xy 137 66) (xy 137 81) (xy 138 82) (xy 143 82) (xy 143 108)
-				(xy 144 109) (xy 148 109) (xy 149 108)
-			)
-		)
+				(xy 149 66) (xy 148 65) (xy 138 65) (xy 137 66) (xy 137 76) (xy 137 81) (xy 138 82) (xy 142 82)
+				(xy 143 83) (xy 143 108) (xy 144 109) (xy 148 109) (xy 149 108)
+			)
+		)
