File: f446re-motor-3ch/f446re-motor-3ch.kicad_sch (KiCad schematic)
At the start: 54 parts, among them J1 電源コネクタ, J2 デバッグ用端子, J3 CANコネクタ, J4 CH1 モータ, J5 CH1 エンコーダ, J6 CH2 モータ, J7 CH2 エンコーダ, J8 CH3 モータ, J9 CH3 エンコーダ, SW1 リセットスイッチ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

Commit message: 2025/02/03/12:25
Parts:
- C12, C13: value C -> 15pF
- renumbered J5 to J4, J4 to J5, J7 to J6, J6 to J7, J9 to J8, J8 to J9
Connections:
- net CAN_RX: now also U1.33 (PB12); no longer U1.44 (PA11)
- net CAN_RX_LED: now also D3.2 (A), U1.39 (PC8); no longer R4.1, U1.14 (PA0)
- net CAN_TX: now also U1.34 (PB13); no longer U1.45 (PA12)
- net CAN_TX_LED: now also D2.2 (A), U1.40 (PC9); no longer R3.1, U1.15 (PA1)
- net CH2_MOTOR_DIR: now also U1.35 (PB14); no longer U1.33 (PB12)
- net GND: now also R3.1, R4.1; no longer D2.1 (K), D3.1 (K)
- net at R3.2: now also D2.1 (K); no longer D2.2 (A)
- net at R4.2: now also D3.1 (K); no longer D3.2 (A)
- net CAN_H renamed CAN+
- net CAN_L renamed CAN-
Other:
- moved on the sheet: D2, D3, R3, R4
Changed lines of the file:
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@@
 	)
 	(no_connect
-		(at 138.43 128.27)
+		(at 138.43 92.71)
 	)
 	(no_connect
-		(at 97.79 107.95)
+		(at 138.43 128.27)
 	)
 	(no_connect
@@
 	)
 	(no_connect
-		(at 138.43 138.43)
-	)
-	(no_connect
 		(at 138.43 87.63)
 	)
@@
 	)
 	(no_connect
-		(at 138.43 140.97)
+		(at 138.43 62.23)
 	)
 	(no_connect
-		(at 97.79 105.41)
+		(at 138.43 140.97)
 	)
 	(no_connect
@@
 	)
 	(no_connect
-		(at 138.43 135.89)
+		(at 138.43 90.17)
+	)
+	(no_connect
+		(at 138.43 64.77)
 	)
 	(no_connect
@@
 		)
 	)
-	(global_label "CAN_H"
+	(global_label "CAN+"
 		(shape bidirectional)
 		(at 30.48 147.32 0)
@@
 		)
 		(property "Intersheetrefs" "${INTERSHEET_REFS}"
-			(at 40.5637 147.32 0)
+			(at 39.838 147.32 0)
 			(effects
 				(font
@@
 		)
 	)
-	(global_label "CAN_L"
+	(global_label "CAN-"
 		(shape bidirectional)
 		(at 90.17 166.37 0)
@@
 		)
 		(property "Intersheetrefs" "${INTERSHEET_REFS}"
-			(at 99.9513 166.37 0)
+			(at 99.528 166.37 0)
 			(effects
 				(font
@@
 	(global_label "CAN_RX"
 		(shape input)
-		(at 138.43 90.17 0)
+		(at 138.43 133.35 0)
 		(fields_autoplaced yes)
 		(effects
@@
 		)
 		(property "Intersheetrefs" "${INTERSHEET_REFS}"
-			(at 148.5514 90.17 0)
+			(at 148.5514 133.35 0)
 			(effects
 				(font
@@
 	(global_label "CH2_MOTOR_DIR"
 		(shape output)
-		(at 138.43 133.35 0)
+		(at 138.43 138.43 0)
 		(fields_autoplaced yes)
 		(effects
@@
 		)
 		(property "Intersheetrefs" "${INTERSHEET_REFS}"
-			(at 156.6552 133.35 0)
+			(at 156.6552 138.43 0)
 			(effects
 				(font
@@
 	(global_label "CAN_TX"
 		(shape output)
-		(at 138.43 92.71 0)
+		(at 138.43 135.89 0)
 		(fields_autoplaced yes)
 		(effects
@@
 		)
 		(property "Intersheetrefs" "${INTERSHEET_REFS}"
-			(at 148.249 92.71 0)
+			(at 148.249 135.89 0)
 			(effects
 				(font
@@
 		)
 	)
-	(global_label "CAN_L"
+	(global_label "CAN-"
 		(shape bidirectional)
 		(at 30.48 149.86 0)
@@
 		)
 		(property "Intersheetrefs" "${INTERSHEET_REFS}"
-			(at 40.2613 149.86 0)
+			(at 39.838 149.86 0)
 			(effects
 				(font
@@
 	(global_label "CAN_TX_LED"
 		(shape output)
-		(at 138.43 64.77 0)
+		(at 97.79 107.95 180)
 		(fields_autoplaced yes)
 		(effects
@@
 				(size 1.27 1.27)
 			)
-			(justify left)
+			(justify right)
 		)
 		(property "Intersheetrefs" "${INTERSHEET_REFS}"
-			(at 152.6637 64.77 0)
+			(at 83.5563 107.95 0)
 			(effects
 				(font
 					(size 1.27 1.27)
 				)
-				(justify left)
+				(justify right)
 				(hide yes)
 			)
@@
 		)
 	)
-	(global_label "CAN_H"
+	(global_label "CAN+"
 		(shape bidirectional)
 		(at 90.17 161.29 0)
@@
 		)
 		(property "Intersheetrefs" "${INTERSHEET_REFS}"
-			(at 100.2537 161.29 0)
+			(at 99.528 161.29 0)
 			(effects
 				(font
@@
 	(global_label "CAN_RX_LED"
 		(shape output)
-		(at 138.43 62.23 0)
+		(at 97.79 105.41 180)
 		(fields_autoplaced yes)
 		(effects
@@
 				(size 1.27 1.27)
 			)
-			(justify left)
+			(justify right)
 		)
 		(property "Intersheetrefs" "${INTERSHEET_REFS}"
-			(at 152.9661 62.23 0)
+			(at 83.2539 105.41 0)
 			(effects
 				(font
 					(size 1.27 1.27)
 				)
-				(justify left)
+				(justify right)
 				(hide yes)
 			)
@@
 	(symbol
 		(lib_id "Device:R")
-		(at 60.96 111.76 0)
+		(at 60.96 121.92 180)
 		(unit 1)
 		(exclude_from_sim no)
@@
 		(fields_autoplaced yes)
 		(property "Reference" "R3"
-			(at 63.5 110.4899 0)
+			(at 63.5 120.6499 0)
 			(effects
 				(font
 					(size 1.27 1.27)
 				)
-				(justify left)
+				(justify right)
 			)
 		)
 		(property "Value" "200Ω"
-			(at 63.5 113.0299 0)
+			(at 63.5 123.1899 0)
 			(effects
 				(font
 					(size 1.27 1.27)
 				)
-				(justify left)
+				(justify right)
 			)
 		)
 		(property "Footprint" "Resistor_SMD:R_0603_1608Metric"
-			(at 59.182 111.76 90)
+			(at 62.738 121.92 90)
 			(effects
 				(font
@@
 		)
 		(property "Datasheet" "~"
-			(at 60.96 111.76 0)
+			(at 60.96 121.92 0)
 			(effects
 				(font
@@
 		)
 		(property "Description" "Resistor"
-			(at 60.96 111.76 0)
+			(at 60.96 121.92 0)
 			(effects
 				(font
@@
 			)
 		)
-		(property "Value" "C"
+		(property "Value" "15pF"
 			(at 67.31 74.93 90)
 			(effects
@@
 		(on_board yes)
 		(dnp no)
-		(property "Reference" "J8"
+		(property "Reference" "J9"
 			(at 215.138 130.302 0)
 			(effects
@@
 			(project "f446re-motor-3ch"
 				(path "/8a05aa10-9bb4-4bec-8e67-331108dc97a9"
-					(reference "J8")
+					(reference "J9")
 					(unit 1)
 				)
@@
 		(on_board yes)
 		(dnp no)
-		(property "Reference" "J4"
+		(property "Reference" "J5"
 			(at 215.138 59.182 0)
 			(effects
@@
 			(project ""
 				(path "/8a05aa10-9bb4-4bec-8e67-331108dc97a9"
-					(reference "J4")
+					(reference "J5")
 					(unit 1)
 				)
@@
 		(on_board yes)
 		(dnp no)
-		(property "Reference" "J7"
+		(property "Reference" "J6"
 			(at 272.288 89.662 0)
 			(effects
@@
 			(project "f446re-motor-3ch"
 				(path "/8a05aa10-9bb4-4bec-8e67-331108dc97a9"
-					(reference "J7")
+					(reference "J6")
 					(unit 1)
 				)
@@
 	(symbol
 		(lib_id "Device:LED")
-		(at 60.96 121.92 90)
+		(at 60.96 111.76 90)
 		(unit 1)
 		(exclude_from_sim no)
@@
 		(fields_autoplaced yes)
 		(property "Reference" "D2"
-			(at 64.77 122.2374 90)
+			(at 64.77 112.0774 90)
 			(effects
 				(font
@@
 		)
 		(property "Value" "LED"
-			(at 64.77 124.7774 90)
+			(at 64.77 114.6174 90)
 			(effects
 				(font
@@
 		)
 		(property "Footprint" "LED_SMD:LED_0603_1608Metric"
-			(at 60.96 121.92 0)
+			(at 60.96 111.76 0)
 			(effects
 				(font
@@
 		)
 		(property "Datasheet" "~"
-			(at 60.96 121.92 0)
+			(at 60.96 111.76 0)
 			(effects
 				(font
@@
 		)
 		(property "Description" "Light emitting diode"
-			(at 60.96 121.92 0)
+			(at 60.96 111.76 0)
 			(effects
 				(font
@@
 			)
 		)
-		(property "Value" "C"
+		(property "Value" "15pF"
 			(at 67.31 62.23 90)
 			(effects
@@
 		)
 		(pin "33"
+			(alternate "CAN2_RX")
 		)
 		(pin "51"
@@
 		)
 		(pin "34"
+			(alternate "CAN2_TX")
 		)
 		(pin "25"
@@
 	(symbol
 		(lib_id "Device:LED")
-		(at 71.12 121.92 90)
+		(at 71.12 111.76 90)
 		(unit 1)
 		(exclude_from_sim no)
@@
 		(fields_autoplaced yes)
 		(property "Reference" "D3"
-			(at 74.93 122.2374 90)
+			(at 74.93 112.0774 90)
 			(effects
 				(font
@@
 		)
 		(property "Value" "LED"
-			(at 74.93 124.7774 90)
+			(at 74.93 114.6174 90)
 			(effects
 				(font
@@
 		)
 		(property "Footprint" "LED_SMD:LED_0603_1608Metric"
-			(at 71.12 121.92 0)
+			(at 71.12 111.76 0)
 			(effects
 				(font
@@
 		)
 		(property "Datasheet" "~"
-			(at 71.12 121.92 0)
+			(at 71.12 111.76 0)
 			(effects
 				(font
@@
 		)
 		(property "Description" "Light emitting diode"
-			(at 71.12 121.92 0)
+			(at 71.12 111.76 0)
 			(effects
 				(font
@@
 		(on_board yes)
 		(dnp no)
-		(property "Reference" "J9"
+		(property "Reference" "J8"
 			(at 272.288 125.222 0)
 			(effects
@@
 			(project "f446re-motor-3ch"
 				(path "/8a05aa10-9bb4-4bec-8e67-331108dc97a9"
-					(reference "J9")
+					(reference "J8")
 					(unit 1)
 				)
@@
 		(on_board yes)
 		(dnp no)
-		(property "Reference" "J5"
+		(property "Reference" "J4"
 			(at 272.288 54.102 0)
 			(effects
@@
 			(project ""
 				(path "/8a05aa10-9bb4-4bec-8e67-331108dc97a9"
-					(reference "J5")
+					(reference "J4")
 					(unit 1)
 				)
@@
 		(on_board yes)
 		(dnp no)
-		(property "Reference" "J6"
+		(property "Reference" "J7"
 			(at 215.138 94.742 0)
 			(effects
@@
 			(project "f446re-motor-3ch"
 				(path "/8a05aa10-9bb4-4bec-8e67-331108dc97a9"
-					(reference "J6")
+					(reference "J7")
 					(unit 1)
 				)
@@
 	(symbol
 		(lib_id "Device:R")
-		(at 71.12 111.76 0)
+		(at 71.12 121.92 180)
 		(unit 1)
 		(exclude_from_sim no)
@@
 		(fields_autoplaced yes)
 		(property "Reference" "R4"
-			(at 73.66 110.4899 0)
+			(at 73.66 120.6499 0)
 			(effects
 				(font
 					(size 1.27 1.27)
 				)
-				(justify left)
+				(justify right)
 			)
 		)
 		(property "Value" "200Ω"
-			(at 73.66 113.0299 0)
+			(at 73.66 123.1899 0)
 			(effects
 				(font
 					(size 1.27 1.27)
 				)
-				(justify left)
+				(justify right)
 			)
 		)
 		(property "Footprint" "Resistor_SMD:R_0603_1608Metric"
-			(at 69.342 111.76 90)
+			(at 72.898 121.92 90)
 			(effects
 				(font
@@
 		)
 		(property "Datasheet" "~"
-			(at 71.12 111.76 0)
+			(at 71.12 121.92 0)
 			(effects
 				(font
@@
 		)
 		(property "Description" "Resistor"
-			(at 71.12 111.76 0)
+			(at 71.12 121.92 0)
 			(effects
 				(font
