File: 3ch-motor-control/3ch-motor-control.kicad_pcb (KiCad board)
At the start: 2 copper layers, 75 x 70 mm, 66 parts, among them J1 電源コネクタ, J2 デバッグ端子, J3 CANコネクタ, SW1 リセットスイッチ, U1 AZ1117-3.3, U2 STM32F446RETx, U3 MCP2562-E-SN, Y1 16MHz

Commit message: 2025/02/19/09:55
Routing:
- net GND: vias 138 -> 141
