File: 3omni-control/3omni-control.kicad_pcb (KiCad board)
At the start: 2 copper layers, 75 x 70 mm, 67 parts, among them J1 電源コネクタ, J2 デバッグ端子, J3 CANコネクタ, SW1 リセットスイッチ, U1 AZ1117-3.3, U2 STM32F446RETx, U3 MCP2562-E-SN, Y1 16MHz

Commit message: feat: モータ制御基盤にダイオードを追加。オムニ制御基盤を追加
Other:
- board text added: "3OmniControl v1.0.0 @netetra07"
- board text removed: "MotrorControl 3ch v1.0.1 @netetra07"
Changed lines of the file:
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@@
 		(layer "Edge.Cuts")
 	)
-	(gr_text "MotrorControl 3ch\nv1.0.1\n@netetra07"
+	(gr_text "3OmniControl\nv1.0.0\n@netetra07"
 		(at 100 47 0)
 		(layer "F.SilkS")
