File: f446re-template/f446re-template.kicad_pcb (KiCad board)
At the start: 2 copper layers, 70 x 70 mm, 36 parts, among them J1 電源コネクタ, J2 デバッグ端子, J3 CANコネクタ, SW1 リセットスイッチ, U1 AZ1117-3.3, U2 STM32F446RETx, U3 MCP2562-E-SN, Y1 16MHz

Commit message: 2025/02/08/19:35
Parts:
- C10: moved to B.Cu
- R1: value ???Ω -> 1kΩ
- R2, R3: value 200Ω -> 1kΩ
- moved C10 22.6 mm to (127.5, 78.0)
- moved SW1 1.12 mm to (99.0, 86.0)
- moved C11 0.45 mm to (132.0, 81.2)
- turned D1 to 180 degrees
- turned D2 to 180 degrees
- turned D3 to 180 degrees
- turned R1 to 180 degrees
- turned R2 to 180 degrees
- turned R3 to 180 degrees
Routing:
- net NRST: track 55.4 -> 52.5 mm, vias 0 -> 1
- net +5V: track 66.5 -> 68.5 mm
- net +3.3V: track 148.7 -> 150.3 mm
- net CAN_TX_LED: track 35.7 -> 34.7 mm
- net CAN_RX_LED: track 30.5 -> 29.5 mm
- net GND: track 19.1 -> 19.2 mm, vias 103 -> 122

Commit message: 2025/02/08/20:30
Routing:
- net GND: vias 122 -> 121

Commit message: 2025/02/15/20:27
Parts:
- moved C2 12.9 mm to (111.7, 87.3), turned to 180 degrees
- moved C1 5.71 mm to (114.0, 98.7), turned to 180 degrees
- moved U1 3.45 mm to (112.5, 93.0), turned to 90 degrees
- moved D1 2.50 mm to (102.5, 107.0)
- moved D2 2.50 mm to (107.5, 107.0)
- moved D3 2.50 mm to (112.5, 107.0)
- moved R1 2.50 mm to (102.5, 104.0)
- moved R2 2.50 mm to (107.5, 104.0)
- moved R3 2.50 mm to (112.5, 104.0)
Routing:
- net +5V: track 68.5 -> 76.1 mm
- net +3.3V: track 150.3 -> 149.2 mm
- net CAN_TX: track 20.6 -> 21.3 mm
- net CAN_RX: track 24.7 -> 25.3 mm
- net CAN_RX_LED: track 29.5 -> 28.8 mm
- net CAN_TX_LED: track 34.7 -> 34.1 mm
- net GND: track 19.2 -> 19.1 mm, vias 121 -> 99
Other:
- board text added: "template v1.0.0 @xxxxxxxx"

Commit message: 2025/06/09/23:25
Parts:
- added D4: D_Schottky, my_library:US2H, F.Cu at (113.8, 98.0)
- added D5: D_Schottky, my_library:US2H, F.Cu at (109.7, 100.8)
- moved C1 1.55 mm to (114.8, 100.0), turned to -90 degrees
- moved C2 1.10 mm to (111.7, 86.2)
- moved U1 1.10 mm to (112.5, 91.9)
Connections:
- J1 pad 2: +5V -> Net-(D5-A)
Routing:
- net +3.3V: track 149.2 -> 151.9 mm
- net +5V: track 76.1 -> 77.0 mm, vias 1 -> 2
